File: Kicad/mowgli_PCB.kicad_pcb (KiCad board)
At the start: 2 copper layers, 65 x 56 mm, 24 parts, among them J1 GPIO, J18 ZX-HY2.0-9PZZ, J3 MPU-6050, J7 Conn_01x03

Commit message: Correction inversion des pin 4 et 6 de J18
Parts:
- removed J3: MPU-6050, xtech:GY-521
- added J5: MPU-6050, xtech:GY-521, F.Cu at (145.7, 70.9)
- GPIO18, GPIO19: value Conn_01x03 -> ZX-HY2.0-3P
- GPS1: value ~ -> UM98x
- I2C_1, UART0, UART2, UART3, UART4: value Conn_01x04 -> ZX-HY2.0-4P
- J7: value Conn_01x03 -> TerminalBloc_P2.54mm_Horizontal
Connections:
- J18 pad 4: +5V_MB -> Net-(J18-Pin_4)
- J18 pad 6: Net-(J18-Pin_6) -> +5V_MB
Routing:
- net Net-(J18-Pin_4): track 0.00 -> 18.8 mm
- net Net-(J18-Pin_6): track 14.6 -> 0.00 mm
- net +5V_MB: track 10.6 -> 8.91 mm, vias 0 -> 2
