File: Kicad/mowgli_PCB.kicad_sch (KiCad schematic)
At the start: 20 parts, among them J1 GPIO, J18 ZX-HY2.0-9PZZ, J3 MPU-6050, J7 TerminalBloc_P2.54mm_Horizont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

Commit message: Correction inversion des pin 4 et 6 de J18
Parts:
- renumbered J3 to J5
Connections:
- net +5V_MB: now also J18.6 (Pin_6); no longer J18.4 (Pin_4)
- net at J5.4 (Pin_4): now also J18.4 (Pin_4); no longer J18.6 (Pin_6)
Changed lines of the file:
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@@
 	(wire
 		(pts
-			(xy 226.06 125.73) (xy 226.06 138.43)
-		)
-		(stroke
-			(width 0)
-			(type default)
-		)
-	)
-	(wire
-		(pts
 			(xy 256.54 118.11) (xy 254 118.11)
 		)
@@
 	(wire
 		(pts
+			(xy 228.6 140.97) (xy 256.54 140.97)
+		)
+		(stroke
+			(width 0)
+			(type default)
+		)
+	)
+	(wire
+		(pts
 			(xy 163.83 66.04) (xy 163.83 71.12)
 		)
@@
 	(wire
 		(pts
+			(xy 219.71 135.89) (xy 256.54 135.89)
+		)
+		(stroke
+			(width 0)
+			(type default)
+		)
+	)
+	(wire
+		(pts
 			(xy 207.01 41.91) (xy 207.01 48.26)
 		)
@@
 	(wire
 		(pts
-			(xy 228.6 135.89) (xy 256.54 135.89)
+			(xy 200.66 125.73) (xy 231.14 125.73)
 		)
 		(stroke
@@
 	(wire
 		(pts
-			(xy 219.71 140.97) (xy 219.71 128.27)
-		)
-		(stroke
-			(width 0)
-			(type default)
-		)
-	)
-	(wire
-		(pts
 			(xy 76.2 27.94) (xy 73.66 27.94)
 		)
@@
 	(wire
 		(pts
+			(xy 231.14 138.43) (xy 231.14 125.73)
+		)
+		(stroke
+			(width 0)
+			(type default)
+		)
+	)
+	(wire
+		(pts
 			(xy 81.28 116.84) (xy 81.28 124.46)
 		)
@@
 	(wire
 		(pts
-			(xy 228.6 109.22) (xy 228.6 135.89)
+			(xy 228.6 109.22) (xy 228.6 140.97)
 		)
 		(stroke
@@
 	(wire
 		(pts
+			(xy 219.71 135.89) (xy 219.71 128.27)
+		)
+		(stroke
+			(width 0)
+			(type default)
+		)
+	)
+	(wire
+		(pts
 			(xy 231.14 34.29) (xy 237.49 34.29)
 		)
@@
 	(wire
 		(pts
+			(xy 231.14 138.43) (xy 256.54 138.43)
+		)
+		(stroke
+			(width 0)
+			(type default)
+		)
+	)
+	(wire
+		(pts
 			(xy 209.55 148.59) (xy 209.55 123.19)
 		)
@@
 	(wire
 		(pts
-			(xy 226.06 138.43) (xy 256.54 138.43)
-		)
-		(stroke
-			(width 0)
-			(type default)
-		)
-	)
-	(wire
-		(pts
 			(xy 236.22 120.65) (xy 236.22 121.92)
 		)
@@
 	(wire
 		(pts
-			(xy 200.66 125.73) (xy 226.06 125.73)
-		)
-		(stroke
-			(width 0)
-			(type default)
-		)
-	)
-	(wire
-		(pts
-			(xy 219.71 140.97) (xy 256.54 140.97)
-		)
-		(stroke
-			(width 0)
-			(type default)
-		)
-	)
-	(wire
-		(pts
 			(xy 60.96 50.8) (xy 31.75 50.8)
 		)
@@
 		(on_board yes)
 		(dnp no)
-		(property "Reference" "J3"
+		(property "Reference" "J5"
 			(at 193.04 128.2699 0)
 			(effects
@@
 			(project ""
 				(path "/e63e39d7-6ac0-4ffd-8aa3-1841a4541b55"
-					(reference "J3")
+					(reference "J5")
 					(unit 1)
 				)
